File: hardware/power/power.kicad_sch (KiCad schematic)
At the start: 38 parts, among them J2 Conn_01x04_Pin, J4 Conn_01x04_Pin, P1 USB_C_Plug_USB2.0, U2 ESP32-S3-WROOM-1, U4 MCP1825S

Commit message: major changes
Parts:
- removed BT1: Battery_Cell, Connector_AMASS:AMASS_XT30U-M_1x02_P5.0mm_Vertical, symbol Device:Battery_Cell
- removed C13: 4.7n, Capacitor_SMD:C_0402_1005Metric, symbol Device:C
- removed C14: 100n, Capacitor_SMD:C_0402_1005Metric, symbol Device:C
- removed C5, C6: 100p, Capacitor_SMD:C_0402_1005Metric, symbol Device:C
- removed H2: M2.5, MountingHole:MountingHole_2.7mm_M2.5, symbol Mechanical:MountingHole
- removed J2: Conn_01x04_Pin, Connector_PinSocket_2.00mm:PinSocket_1x04_P2.00mm_Vertical, symbol Connector:Conn_01x04_Pin
- removed P1: USB_C_Plug_USB2.0, Connector_USB:USB_C_Receptacle_HRO_TYPE-C-31-M-12, symbol Connector:USB_C_Plug_USB2.0
- removed R1, R2: 22, Resistor_SMD:R_0402_1005Metric, symbol Device:R_US
- removed R3, R4: 60, Resistor_SMD:R_0402_1005Metric, symbol Device:R
- removed U1: ~, Package_SO:SO-8_3.9x4.9mm_P1.27mm, symbol 0_pwrmtr:TCAN334
- added J1: Conn_02x03_Odd_Even, Connector_IDC:IDC-Header_2x03_P2.54mm_Vertical, symbol Connector_Generic:Conn_02x03_Odd_Even
- added J2: Conn_01x02_Pin, Connector_PinHeader_1.27mm:PinHeader_1x02_P1.27mm_Vertical, symbol Connector:Conn_01x02_Pin
- D4: value 1N400X -> D; footprint Diode_THT:D_T-1_P5.08mm_Horizontal -> 0_myfootprints:SD103CW
- J4: footprint Connector_PinSocket_2.00mm:PinSocket_1x04_P2.00mm_Vertical -> Connector_JST:JST_EH_S4B-EH_1x04_P2.50mm_Horizontal
Connections:
- net SHDN_{CAN} is gone; now on net LED_{2}: U2.25 (IO48)
- net STB_{CAN} is gone; now on net LED_{1}: U2.26 (IO45)
- net +3V3: now also J1.2 (Pin_2), J2.1 (Pin_1); no longer J4.1 (Pin_1)
- net GND: now also J1.4 (Pin_4), J2.2 (Pin_2)
- net LED_{1}: no longer U2.35 (IO42)
- net LED_{2}: no longer U2.34 (IO41)
- net RX: now also U2.21 (IO13), J1.5 (Pin_5); no longer U2.24 (IO47)
- net TX: now also U2.22 (IO14), J1.3 (Pin_3); no longer U2.23 (IO21)
- net IO0: now reaches U2.27 (IO0)
- net IO0: now also J1.6 (Pin_6)
- net EN: now reaches U2.3 (EN)
- net EN: now also J1.1 (Pin_1)
- net +5V renamed BATT
- net BATT: now also J4.1 (Pin_1)
- net USB_{D}+: no longer names the net of U2.16 (IO46)
- net USB_{D}-: no longer names the net of U2.17 (IO9)
Other:
- note added: "Programming (ESP PROG)"
- note added: "Wired Power"
- note removed: "Battery Connection (3.7V-5V, XT30)"
- note removed: "CAN + Wired Power Header"
- note removed: "CAN Transceiver (TCAN334GD)"
- moved on the sheet: C11, C12, U4
