File: hardware/rev3/nexus_power_rev3/nexus_power_rev3.kicad_pcb (KiCad board)
At the start: 2 copper layers, 48 x 34.1 mm, 23 parts, among them J1 Conn_02x03_Odd_Even, J2 Conn_01x02_Pin, J4 Conn_01x04_Pin, U1 ADS131M03, U2 ESP32-S3-WROOM-1, U3 ICM-42670-P1

Commit message: Update for resolder
added pull up resistors and changed j2 footprint
Parts:
- added R1: 5.1k, Resistor_SMD:R_0603_1608Metric, F.Cu at (141.6, 94.5)
- added R2: 5.1k, Resistor_SMD:R_0603_1608Metric, F.Cu at (164.1, 105.8)
Routing:
- net +3.3V: track 0.00 -> 28.9 mm, vias 0 -> 2
- net /EN: track 26.0 -> 28.8 mm
- net /IO0: track 12.2 -> 15.0 mm
