File: hardware/rev3/nexus_power_rev3/nexus_power_rev3.kicad_sch (KiCad schematic)
At the start: 23 parts, among them J1 Conn_02x03_Odd_Even, J2 Conn_01x02_Pin, J4 Conn_01x04_Pin, U1 ADS131M03, U2 ESP32-S3-WROOM-1, U3 ICM-42670-P1

Commit message: Update for resolder
added pull up resistors and changed j2 footprint
Parts:
- added R1, R2: 5.1k, Resistor_SMD:R_0603_1608Metric, symbol Device:R
Connections:
- net EN: now also R1.1
- net IO0: now also R2.2
- new net +3.3V: R1.2, R2.1
