File: hardware/rev4/final hpv power.kicad_sch (KiCad schematic)
At the start: 32 parts

Commit message: Final fixes
Connections:
- net at R4.1, U3.7 (INA-): now also C10.2
- net at J2.4 (Pin_4), R4.2: no longer C10.2
- net at J2.3 (Pin_3), R3.1: no longer C10.1
- net at R3.2, U3.8 (INA+): now also C10.1
Other:
- moved on the sheet: C10, R3, R4
Changed lines of the file:
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@@
 	)
 	(junction
-		(at 60.96 21.59)
+		(at 217.17 69.85)
 		(diameter 0)
 		(color 0 0 0 0)
 	)
 	(junction
-		(at 240.03 36.83)
+		(at 217.17 78.74)
 		(diameter 0)
 		(color 0 0 0 0)
 	)
 	(junction
-		(at 127 63.5)
+		(at 60.96 21.59)
 		(diameter 0)
 		(color 0 0 0 0)
 	)
 	(junction
-		(at 73.66 40.64)
+		(at 240.03 36.83)
 		(diameter 0)
 		(color 0 0 0 0)
 	)
 	(junction
-		(at 138.43 63.5)
+		(at 127 63.5)
 		(diameter 0)
 		(color 0 0 0 0)
 	)
 	(junction
-		(at 207.01 78.74)
+		(at 73.66 40.64)
 		(diameter 0)
 		(color 0 0 0 0)
 	)
 	(junction
-		(at 217.17 58.42)
+		(at 138.43 63.5)
 		(diameter 0)
 		(color 0 0 0 0)
 	)
 	(junction
-		(at 207.01 69.85)
+		(at 217.17 58.42)
 		(diameter 0)
 		(color 0 0 0 0)
@@
 	(wire
 		(pts
+			(xy 214.63 78.74) (xy 217.17 78.74)
+		)
+		(stroke
+			(width 0)
+			(type default)
+		)
+	)
+	(wire
+		(pts
 			(xy 255.27 68.58) (xy 257.81 68.58)
 		)
@@
 	(wire
 		(pts
-			(xy 220.98 69.85) (xy 229.87 69.85)
+			(xy 214.63 69.85) (xy 217.17 69.85)
 		)
 		(stroke
@@
 	(wire
 		(pts
+			(xy 217.17 78.74) (xy 220.98 78.74)
+		)
+		(stroke
+			(width 0)
+			(type default)
+		)
+	)
+	(wire
+		(pts
 			(xy 73.66 38.1) (xy 76.2 38.1)
 		)
@@
 	(wire
 		(pts
-			(xy 220.98 72.39) (xy 223.52 72.39)
+			(xy 229.87 69.85) (xy 229.87 68.58)
 		)
 		(stroke
@@
 	(wire
 		(pts
-			(xy 229.87 69.85) (xy 229.87 68.58)
+			(xy 71.12 29.21) (xy 71.12 31.75)
 		)
 		(stroke
@@
 	(wire
 		(pts
-			(xy 71.12 29.21) (xy 71.12 31.75)
+			(xy 111.76 85.09) (xy 115.57 85.09)
 		)
 		(stroke
@@
 	(wire
 		(pts
-			(xy 111.76 85.09) (xy 115.57 85.09)
+			(xy 220.98 72.39) (xy 220.98 78.74)
 		)
 		(stroke
@@
 	(wire
 		(pts
-			(xy 207.01 68.58) (xy 207.01 69.85)
+			(xy 204.47 63.5) (xy 204.47 69.85)
 		)
 		(stroke
@@
 	(wire
 		(pts
-			(xy 213.36 69.85) (xy 207.01 69.85)
+			(xy 207.01 69.85) (xy 204.47 69.85)
 		)
 		(stroke
@@
 	(wire
 		(pts
-			(xy 257.81 78.74) (xy 255.27 78.74)
+			(xy 217.17 69.85) (xy 229.87 69.85)
 		)
 		(stroke
@@
 	(wire
 		(pts
-			(xy 54.61 182.88) (xy 50.8 182.88)
+			(xy 257.81 78.74) (xy 255.27 78.74)
 		)
 		(stroke
@@
 	(wire
 		(pts
-			(xy 199.39 58.42) (xy 205.74 58.42)
+			(xy 54.61 182.88) (xy 50.8 182.88)
 		)
 		(stroke
@@
 	(wire
 		(pts
-			(xy 54.61 162.56) (xy 50.8 162.56)
+			(xy 199.39 58.42) (xy 205.74 58.42)
 		)
 		(stroke
@@
 	(wire
 		(pts
-			(xy 187.96 130.81) (xy 191.77 130.81)
+			(xy 54.61 162.56) (xy 50.8 162.56)
 		)
 		(stroke
@@
 	(wire
 		(pts
-			(xy 207.01 78.74) (xy 213.36 78.74)
+			(xy 187.96 130.81) (xy 191.77 130.81)
 		)
 		(stroke
@@
 	(wire
 		(pts
-			(xy 204.47 68.58) (xy 204.47 63.5)
+			(xy 60.96 29.21) (xy 71.12 29.21)
 		)
 		(stroke
@@
 	(wire
 		(pts
-			(xy 60.96 29.21) (xy 71.12 29.21)
+			(xy 138.43 63.5) (xy 148.59 63.5)
 		)
 		(stroke
@@
 	(wire
 		(pts
-			(xy 138.43 63.5) (xy 148.59 63.5)
+			(xy 223.52 83.82) (xy 229.87 83.82)
 		)
 		(stroke
@@
 	(wire
 		(pts
-			(xy 223.52 83.82) (xy 229.87 83.82)
+			(xy 217.17 77.47) (xy 217.17 78.74)
 		)
 		(stroke
@@
 	(wire
 		(pts
-			(xy 207.01 68.58) (xy 204.47 68.58)
+			(xy 223.52 72.39) (xy 220.98 72.39)
 		)
 		(stroke
@@
 	(wire
 		(pts
-			(xy 213.36 72.39) (xy 213.36 78.74)
-		)
-		(stroke
-			(width 0)
-			(type default)
-		)
-	)
-	(wire
-		(pts
 			(xy 146.05 26.67) (xy 146.05 27.94)
 		)
@@
 	(wire
 		(pts
-			(xy 207.01 77.47) (xy 207.01 78.74)
-		)
-		(stroke
-			(width 0)
-			(type default)
-		)
-	)
-	(wire
-		(pts
 			(xy 146.05 27.94) (xy 140.97 27.94)
 		)
@@
 	(symbol
 		(lib_id "Device:R")
-		(at 217.17 72.39 270)
+		(at 210.82 78.74 270)
 		(unit 1)
 		(exclude_from_sim no)
@@
 		(dnp no)
 		(property "Reference" "R4"
-			(at 217.17 74.422 90)
+			(at 210.82 80.772 90)
 			(effects
 				(font
@@
 		)
 		(property "Value" "100"
-			(at 217.17 70.104 90)
+			(at 210.82 76.454 90)
 			(effects
 				(font
@@
 		)
 		(property "Footprint" "Resistor_SMD:R_0805_2012Metric"
-			(at 217.17 70.612 90)
+			(at 210.82 76.962 90)
 			(effects
 				(font
@@
 		)
 		(property "Datasheet" "https://www.vishay.com/docs/20035/dcrcwe3.pdf"
-			(at 217.17 72.39 0)
+			(at 210.82 78.74 0)
 			(effects
 				(font
@@
 		)
 		(property "Description" "Resistor"
-			(at 217.17 72.39 0)
+			(at 210.82 78.74 0)
 			(effects
 				(font
@@
 		)
 		(property "Digikey Link" "https://www.digikey.ca/en/products/detail/vishay-dale/CRCW0805100RFKEA/1175523"
-			(at 217.17 72.39 90)
+			(at 210.82 78.74 90)
 			(effects
 				(font
@@
 		)
 		(property "Item Name" "Resistor"
-			(at 217.17 72.39 90)
+			(at 210.82 78.74 90)
 			(effects
 				(font
@@
 		)
 		(property "Manufacturer" "  Vishay Dale"
-			(at 217.17 72.39 90)
+			(at 210.82 78.74 90)
 			(effects
 				(font
@@
 		)
 		(property "Part number" "  CRCW0805100RFKEA"
-			(at 217.17 72.39 90)
+			(at 210.82 78.74 90)
 			(effects
 				(font
@@
 		)
 		(instances
-			(project "HPV crank power meter"
+			(project "final hpv power"
 				(path "/27234012-9449-4b0c-98e8-e6a5c387b255"
 					(reference "R4")
@@
 	(symbol
 		(lib_id "Device:R")
-		(at 217.17 69.85 90)
+		(at 210.82 69.85 90)
 		(unit 1)
 		(exclude_from_sim no)
@@
 		(dnp no)
 		(property "Reference" "R3"
-			(at 216.662 67.818 90)
+			(at 210.312 67.818 90)
 			(effects
 				(font
@@
 		)
 		(property "Value" "100"
-			(at 217.17 72.39 90)
+			(at 210.82 72.39 90)
 			(effects
 				(font
@@
 		)
 		(property "Footprint" "Resistor_SMD:R_0805_2012Metric"
-			(at 217.17 71.628 90)
+			(at 210.82 71.628 90)
 			(effects
 				(font
@@
 		)
 		(property "Datasheet" "https://www.vishay.com/docs/20035/dcrcwe3.pdf"
-			(at 217.17 69.85 0)
+			(at 210.82 69.85 0)
 			(effects
 				(font
@@
 		)
 		(property "Description" "Resistor"
-			(at 217.17 69.85 0)
+			(at 210.82 69.85 0)
 			(effects
 				(font
@@
 		)
 		(property "Digikey Link" "https://www.digikey.ca/en/products/detail/vishay-dale/CRCW0805100RFKEA/1175523"
-			(at 217.17 69.85 90)
+			(at 210.82 69.85 90)
 			(effects
 				(font
@@
 		)
 		(property "Item Name" "Resistor"
-			(at 217.17 69.85 90)
+			(at 210.82 69.85 90)
 			(effects
 				(font
@@
 		)
 		(property "Manufacturer" "  Vishay Dale"
-			(at 217.17 69.85 90)
+			(at 210.82 69.85 90)
 			(effects
 				(font
@@
 		)
 		(property "Part number" "  CRCW0805100RFKEA"
-			(at 217.17 69.85 90)
+			(at 210.82 69.85 90)
 			(effects
 				(font
@@
 		)
 		(instances
-			(project "HPV crank power meter"
+			(project "final hpv power"
 				(path "/27234012-9449-4b0c-98e8-e6a5c387b255"
 					(reference "R3")
@@
 	(symbol
 		(lib_id "Device:C")
-		(at 207.01 73.66 0)
+		(at 217.17 73.66 0)
 		(unit 1)
 		(exclude_from_sim no)
@@
 		(dnp no)
 		(property "Reference" "C10"
-			(at 205.74 81.026 0)
+			(at 215.9 81.026 0)
 			(effects
 				(font
@@
 		)
 		(property "Value" "0.1u"
-			(at 205.74 83.566 0)
+			(at 215.9 83.566 0)
 			(effects
 				(font
@@
 		)
 		(property "Footprint" "Capacitor_SMD:C_0805_2012Metric"
-			(at 207.9752 77.47 0)
+			(at 218.1352 77.47 0)
 			(effects
 				(font
@@
 		)
 		(property "Datasheet" "https://yageogroup.com/content/datasheet/asset/file/KEM_C1002_X7R_SMD"
-			(at 207.01 73.66 0)
+			(at 217.17 73.66 0)
 			(effects
 				(font
@@
 		)
 		(property "Description" "Unpolarized capacitor"
-			(at 207.01 73.66 0)
+			(at 217.17 73.66 0)
 			(effects
 				(font
@@
 		)
 		(property "Digikey Link" "https://www.digikey.ca/en/products/detail/kemet/C0805C104K5RACTU/411169 "
-			(at 207.01 73.66 0)
+			(at 217.17 73.66 0)
 			(effects
 				(font
@@
 		)
 		(property "Item Name" "Capacitor"
-			(at 207.01 73.66 0)
+			(at 217.17 73.66 0)
 			(effects
 				(font
@@
 		)
 		(property "Manufacturer" "  KEMET"
-			(at 207.01 73.66 0)
+			(at 217.17 73.66 0)
 			(effects
 				(font
@@
 		)
 		(property "Part number" "  C0805C104K5RACTU"
-			(at 207.01 73.66 0)
+			(at 217.17 73.66 0)
 			(effects
 				(font
@@
 		)
 		(instances
-			(project "HPV crank power meter"
+			(project "final hpv power"
 				(path "/27234012-9449-4b0c-98e8-e6a5c387b255"
 					(reference "C10")
