File: hardware/rev4/final hpv power.kicad_pcb (KiCad board)
At the start: 2 copper layers, 39.2 x 44.1 mm, 32 parts

Commit message: Added board maker name
Other:
- board text added: "Nexus Power Rev4"
Changed lines of the file:
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@@
 			(psa4output no)
 			(plot_black_and_white yes)
+			(plotinvisibletext no)
 			(sketchpadsonfab no)
 			(plotpadnumbers no)
@@
 		(layer "Edge.Cuts")
 	)
+	(gr_text "Nexus Power Rev4"
+		(at 119.38 118.11 0)
+		(layer "F.SilkS" knockout)
+		(effects
+			(font
+				(size 1 1)
+				(thickness 0.2)
+				(bold yes)
+			)
+			(justify left bottom)
+		)
+	)
 	(segment
