File: hardware/rev5/rev5.kicad_sch (KiCad schematic)
At the start: 25 parts, among them J3 Conn_02x03_Odd_Even, J4 Conn_01x05, J5 Conn_01x02

Commit message: UPDATE HEADER
Parts:
- J4: footprint Connector_JST:JST_EH_B5B-EH-A_1x05_P2.50mm_Vertical -> Connector_JST:JST_XH_B5B-XH-A_1x05_P2.50mm_Vertical
Changed lines of the file:
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@@
 			)
 		)
-		(property "Footprint" "Connector_JST:JST_EH_B5B-EH-A_1x05_P2.50mm_Vertical"
+		(property "Footprint" "Connector_JST:JST_XH_B5B-XH-A_1x05_P2.50mm_Vertical"
 			(at 180.34 120.65 0)
 			(effects

Commit message: Rev 5 changes
Parts:
- removed J1: ~, Connector_JST:JST_EH_B12B-EH-A_1x12_P2.50mm_Vertical, symbol Connector_Generic:Conn_01x12
- removed J2: ~, Connector_USB:USB_C_Receptacle_GCT_USB4110, symbol Connector:USB_C_Receptacle_USB2.0_14P
- removed R4, R5: 5.1k, Resistor_SMD:R_0805_2012Metric, symbol Device:R
- added J6: USB_C_Receptacle_USB2.0_16P, Connector_USB:USB_C_Receptacle_JAE_DX07S016JA1R1500, symbol Connector:USB_C_Receptacle_USB2.0_16P
- added R6: 5k, Resistor_SMD:R_0805_2012Metric_Pad1.20x1.40mm_HandSolder, symbol Device:R
- added R7, R8: 5.1k, Resistor_SMD:R_0805_2012Metric, symbol Device:R
- added SW1, SW2: SW_Push, Button_Switch_SMD:SW_SPST_SKQG_WithStem, symbol Switch:SW_Push
- added U3: USBLC6-2SC6, Package_TO_SOT_SMD:SOT-23-6, symbol Power_Protection:USBLC6-2SC6
- J4: footprint Connector_JST:JST_XH_B5B-XH-A_1x05_P2.50mm_Vertical -> Connector_JST:JST_XH_S5B-XH-A-1_1x05_P2.50mm_Horizontal
Connections:
- net VCC is gone; now on net +3.3V: J4.2 (Pin_2)
- net VDD is gone; now on net +3.3V: J4.1 (Pin_1)
- net +3.3V: now also R3.1, R6.1; no longer R3.2
- net +5V_USB: now also J6.A4 (VBUS), J6.A9 (VBUS), J6.B4 (VBUS), J6.B9 (VBUS), U3.5 (VBUS)
- net D+: now also J6.A6 (D+), J6.B6 (D+), U3.1 (I/O1), U3.6 (I/O1)
- net D-: now also J6.A7 (D-), J6.B7 (D-), U3.3 (I/O2), U3.4 (I/O2)
- net EN: now also R3.2, SW1.1; no longer R3.1
- net GND: now also J6.A1 (GND), J6.A12 (GND), J6.B1 (GND), J6.B12 (GND), J6.S1 (SHIELD), R7.2, R8.2, SW1.2, SW2.2, U3.2 (GND)
- net GPIO10: no longer names the net of U1.33 (IO40)
- net GPIO9: no longer names the net of U1.34 (IO41)
- net IO0 renamed BOOT
- net BOOT: now also R6.2, SW2.1
- new net: J6.A5 (CC1), R7.1
- new net: J6.B5 (CC2), R8.1
- no-connect marks 20 -> 24
Other:
- note added: "Backflow Prevention"
- note added: "ESP PROG Header"
- note added: "HX711 Header"
- note added: "IMU"
- note added: "Lipo Battery Header w/ 3.7 V input"
- note added: "TVS Diode"
- note added: "USB"
- note added: "VCC"
- note added: "VDD"
- note added: "VDD and VCC are both 3.3V"
- note removed: "Gyroscope"
- note removed: "VDD and VCC are both 3.7"
- note removed: "don't connect header"
- note removed: "esp PROG"
- note removed: "hx711"
- note removed: "lipo battery w/ 3.7 V input"
- moved on the sheet: C1, C2, C3, C4, C5, C6, C7, C8, D1, D2, D3, D4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
