File: hardware/rev5/rev5.kicad_pcb (KiCad board)
At the start: 2 copper layers, 39.2 x 44.1 mm, 25 parts, among them J3 Conn_02x03_Odd_Even, J4 Conn_01x05, J5 Conn_01x02

Commit message: Rev 5 changes
Parts:
- removed J1: ~, Connector_JST:JST_EH_B12B-EH-A_1x12_P2.50mm_Vertical
- removed J2: ~, Connector_USB:USB_C_Receptacle_GCT_USB4110
- removed R4, R5: 5.1k, Resistor_SMD:R_0805_2012Metric
- added J6: USB_C_Receptacle_USB2.0_16P, Connector_USB:USB_C_Receptacle_JAE_DX07S016JA1R1500, F.Cu at (138.2, 90.7)
- added R6: 5k, Resistor_SMD:R_0805_2012Metric_Pad1.20x1.40mm_HandSolder, F.Cu at (142.3, 113.5)
- added R7: 5.1k, Resistor_SMD:R_0805_2012Metric, F.Cu at (145.3, 92.4)
- added R8: 5.1k, Resistor_SMD:R_0805_2012Metric, F.Cu at (144.6, 95.5)
- added SW1: SW_Push, Button_Switch_SMD:SW_SPST_SKQG_WithStem, F.Cu at (137.9, 102.0)
- added SW2: SW_Push, Button_Switch_SMD:SW_SPST_SKQG_WithStem, F.Cu at (137.9, 111.1)
- added U3: USBLC6-2SC6, Package_TO_SOT_SMD:SOT-23-6, F.Cu at (144.9, 85.9)
- J4: footprint Connector_JST:JST_EH_B5B-EH-A_1x05_P2.50mm_Vertical -> Connector_JST:JST_XH_S5B-XH-A-1_1x05_P2.50mm_Horizontal
- moved D2 46.2 mm to (161.0, 112.5), turned to 90 degrees
- moved D1 45.6 mm to (157.4, 112.5), turned to 90 degrees
- moved R2 40.0 mm to (161.0, 108.0), turned to -90 degrees
- moved R1 39.3 mm to (157.4, 108.1), turned to -90 degrees
- moved J4 33.9 mm to (150.8, 130.3)
- moved J5 30.8 mm to (139.5, 131.6), turned to 0 degrees
- moved J3 28.2 mm to (157.5, 90.3), turned to 0 degrees
- moved C5 25.9 mm to (154.5, 117.7)
- moved D3 25.1 mm to (150.0, 114.0)
- moved D4 22.9 mm to (143.2, 120.9), turned to -90 degrees
- moved U2 18.5 mm to (148.9, 120.3), turned to -90 degrees
- moved C2 16.6 mm to (137.8, 66.3), turned to 90 degrees
- moved U1 16.5 mm to (149.1, 68.7)
- moved C3 14.8 mm to (135.5, 70.2), turned to -90 degrees
- moved C7 14.6 mm to (142.5, 117.0)
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Connections:
- net /IO0 renamed /BOOT
- J4 pad 1: /VDD -> +3.3V
- J4 pad 2: /VCC -> +3.3V
- R3 pad 1: /EN -> +3.3V
- R3 pad 2: +3.3V -> /EN
- U1 pad 33: /GPIO10 -> unconnected-(U1-IO40-Pad33)
- U1 pad 34: /GPIO9 -> unconnected-(U1-IO41-Pad34)
Routing:
- net +3.3V: track 21.6 -> 120.1 mm, vias 0 -> 3
- net GND: track 79.4 -> 3.28 mm, vias 13 -> 0
- net /EN: track 53.3 -> 0.00 mm, vias 1 -> 0
- net /TX: track 51.8 -> 0.00 mm, vias 2 -> 0
- net /RX: track 47.1 -> 0.00 mm, vias 2 -> 0
- net +5V_USB: track 8.61 -> 42.1 mm, vias 0 -> 4
- net /MISO: track 30.3 -> 0.00 mm, vias 1 -> 0
- net /BOOT: track 25.1 -> 0.00 mm, vias 1 -> 0
- net /INT1 Gyro: track 23.2 -> 0.00 mm, vias 2 -> 0
- net /MOSI: track 22.1 -> 0.00 mm, vias 2 -> 0
- net /CS Gyro: track 22.1 -> 0.00 mm, vias 2 -> 0
- net /SCLK: track 21.8 -> 0.00 mm, vias 1 -> 0
- net /INT2 Gyro: track 15.8 -> 0.00 mm, vias 2 -> 0
- net /HX711 PDSCK: track 15.7 -> 0.00 mm, vias 2 -> 0
- net /HX711 DOUT: track 11.4 -> 0.00 mm, vias 2 -> 0
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- added copper zone on F.Cu, net GND
- removed copper zone on F.Cu, net +3.3V
Other:
- board size 39.2 x 44.1 mm -> 30 x 76.7 mm
- board text removed: "Nexus Power Rev5"

Commit message: wired the pcb
Parts:
- renumbered ICM-42670-P1 to IMU
Routing:
- net /HX711 DOUT: track 0.00 -> 103.9 mm, vias 0 -> 2
- net /HX711 PDSCK: track 0.00 -> 82.0 mm, vias 0 -> 2
- net /LED: track 0.00 -> 63.8 mm, vias 0 -> 2
- net /EN: track 0.00 -> 62.3 mm, vias 0 -> 3
- net /BOOT: track 0.00 -> 52.6 mm, vias 0 -> 2
- net GND: track 3.28 -> 33.6 mm, vias 0 -> 6
- net /TX: track 0.00 -> 30.0 mm, vias 0 -> 2
- net /RX: track 0.00 -> 29.8 mm
- net /INT2 Gyro: track 0.00 -> 22.6 mm
- net /INT1 Gyro: track 0.00 -> 22.0 mm
- net /D-: track 0.00 -> 21.7 mm
- net /D+: track 0.00 -> 21.7 mm
- net /CS Gyro: track 0.00 -> 21.0 mm
- net /SCLK: track 0.00 -> 20.6 mm
- net /MOSI: track 0.00 -> 20.3 mm
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
Commit message: small changes to the traces
Routing:
- net GND: track 33.6 -> 13.4 mm, vias 6 -> 3
Changed lines of the file:
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@@
-	)
-	(segment
-		(start 140.8744 85.6256)
-		(end 141 85.5)
-		(width 0.25)
-		(layer "F.Cu")
-		(net 28)
 	)
 	(segment
@@
 		(start 135.4594 65.7848)
 		(end 135.4442 65.7696)
-		(width 0.25)
-		(layer "F.Cu")
-		(net 28)
-	)
-	(segment
-		(start 146.2513 91.2487)
-		(end 146.5 91)
-		(width 0.25)
-		(layer "F.Cu")
-		(net 28)
-	)
-	(segment
-		(start 154.343413 94.343413)
-		(end 155.5 95.5)
-		(width 0.25)
-		(layer "F.Cu")
-		(net 28)
-	)
-	(segment
-		(start 146.765 94.2537)
-		(end 144.6022 96.4165)
 		(width 0.25)
 		(layer "F.Cu")
@@
 	)
 	(segment
-		(start 146.2513 92.3798)
-		(end 146.2513 91.2487)
-		(width 0.25)
-		(layer "F.Cu")
-		(net 28)
-	)
-	(segment
 		(start 149.0761 102.0761)
 		(end 149 102)
@@
 	)
 	(segment
-		(start 146.2513 92.3798)
-		(end 146.765 92.8935)
-		(width 0.25)
-		(layer "F.Cu")
-		(net 28)
-	)
-	(segment
 		(start 149.5761 102.9094)
 		(end 149.0761 102.9094)
-		(width 0.25)
-		(layer "F.Cu")
-		(net 28)
-	)
-	(segment
-		(start 140.8744 86.3822)
-		(end 140.8744 85.6256)
 		(width 0.25)
 		(layer "F.Cu")
@@
 		(net 28)
 	)
-	(segment
-		(start 154.343413 91.343413)
-		(end 154.343413 94.343413)
-		(width 0.25)
-		(layer "F.Cu")
-		(net 28)
-	)
-	(segment
-		(start 146.765 92.8935)
-		(end 146.765 94.2537)
-		(width 0.25)
-		(layer "F.Cu")
-		(net 28)
-	)
-	(via
-		(at 141 85.5)
-		(size 0.6)
-		(drill 0.3)
-		(layers "F.Cu" "B.Cu")
-		(net 28)
-	)
 	(via
 		(at 155.5 95.5)
-		(size 0.6)
-		(drill 0.3)
-		(layers "F.Cu" "B.Cu")
-		(net 28)
-	)
-	(via
-		(at 154.343413 91.343413)
 		(size 0.6)
 		(drill 0.3)
@@
 		(drill 0.3)
 		(layers "F.Cu" "B.Cu")
-		(net 28)
-	)
-	(via
-		(at 146.5 91)
-		(size 0.6)
-		(drill 0.3)
-		(layers "F.Cu" "B.Cu")
-		(net 28)
-	)
-	(segment
-		(start 154 91)
-		(end 154.343413 91.343413)
-		(width 0.25)
-		(layer "B.Cu")
 		(net 28)
 	)
@@
 		(width 0.25)
 		(layer "B.Cu")
-		(net 28)
-	)
-	(segment
-		(start 146.5 91)
-		(end 154 91)
-		(width 0.25)
-		(layer "B.Cu")

Commit message: fixed header traces
Routing:
- net /TX: track 30.0 -> 27.3 mm, vias 2 -> 1
- net /BOOT: track 52.6 -> 52.9 mm, vias 2 -> 1
- net /EN: vias 3 -> 2
Changed lines of the file:
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@@
-	)
-	(segment
-		(start 160.0822 97.4178)
-		(end 160 97.5)
-		(width 0.15)
-		(layer "F.Cu")
-		(net 3)
 	)
 	(segment
@@
 	)
 	(segment
-		(start 160.0822 95.4012)
-		(end 160.0822 97.4178)
-		(width 0.15)
-		(layer "F.Cu")
-		(net 3)
-	)
-	(segment
 		(start 139.717 107.9742)
 		(end 139.717 114.1742)
@@
 	)
 	(via
-		(at 160 97.5)
+		(at 141 108)
 		(size 0.6)
 		(drill 0.3)
@@
 		(net 3)
 	)
-	(via
-		(at 141 108)
-		(size 0.6)
-		(drill 0.3)
-		(layers "F.Cu" "B.Cu")
-		(net 3)
-	)
-	(segment
-		(start 149.5 108)
-		(end 160 97.5)
+	(segment
+		(start 160.5 95.819)
+		(end 160.0822 95.4012)
 		(width 0.15)
 		(layer "B.Cu")
@@
 	)
 	(segment
+		(start 160.5 97)
+		(end 160.5 95.819)
+		(width 0.15)
+		(layer "B.Cu")
+		(net 3)
+	)
+	(segment
+		(start 149.5 108)
+		(end 160.5 97)
+		(width 0.15)
+		(layer "B.Cu")
+		(net 3)
+	)
+	(segment
 		(start 142.760902 91.3538)
 		(end 144.934314 91.3538)
@@
 	)
 	(segment
+		(start 139.7212 98.881)
+		(end 140.881 98.881)
+		(width 0.15)
+		(layer "F.Cu")
+		(net 5)
+	)
+	(segment
+		(start 139.7212 98.881)
+		(end 139.7212 105.081)
+		(width 0.15)
+		(layer "F.Cu")
+		(net 5)
+	)
+	(via
+		(at 141.5 66.5)
+		(size 0.6)
+		(drill 0.3)
+		(layers "F.Cu" "B.Cu")
+		(net 5)
+	)
+	(via
+		(at 141 99)
+		(size 0.6)
+		(drill 0.3)
+		(layers "F.Cu" "B.Cu")
+		(net 5)
+	)
+	(segment
+		(start 147.5 99)
+		(end 141 99)
+		(width 0.15)
+		(layer "B.Cu")
+		(net 5)
+	)
+	(segment
+		(start 141.5 66.5)
+		(end 141.5 71)
+		(width 0.15)
+		(layer "B.Cu")
+		(net 5)
+	)
+	(segment
+		(start 141.5 71)
+		(end 156 85.5)
+		(width 0.15)
+		(layer "B.Cu")
+		(net 5)
+	)
+	(segment
+		(start 157.5422 90.3212)
+		(end 156.1788 90.3212)
+		(width 0.2)
+		(layer "B.Cu")
+		(net 5)
+	)
+	(segment
+		(start 156 90.5)
+		(end 147.5 99)
+		(width 0.15)
+		(layer "B.Cu")
+		(net 5)
+	)
+	(segment
 		(start 156.1788 90.3212)
 		(end 156 90.5)
-		(width 0.15)
-		(layer "F.Cu")
-		(net 5)
-	)
-	(segment
-		(start 139.7212 98.881)
-		(end 140.881 98.881)
-		(width 0.15)
-		(layer "F.Cu")
-		(net 5)
-	)
-	(segment
-		(start 139.7212 98.881)
-		(end 139.7212 105.081)
-		(width 0.15)
-		(layer "F.Cu")
-		(net 5)
-	)
-	(segment
-		(start 157.5422 90.3212)
-		(end 156.1788 90.3212)
-		(width 0.15)
-		(layer "F.Cu")
-		(net 5)
-	)
-	(via
-		(at 156 90.5)
-		(size 0.6)
-		(drill 0.3)
-		(layers "F.Cu" "B.Cu")
-		(net 5)
-	)
-	(via
-		(at 141.5 66.5)
-		(size 0.6)
-		(drill 0.3)
-		(layers "F.Cu" "B.Cu")
-		(net 5)
-	)
-	(via
-		(at 141 99)
-		(size 0.6)
-		(drill 0.3)
-		(layers "F.Cu" "B.Cu")
-		(net 5)
-	)
-	(segment
-		(start 147.5 99)
-		(end 141 99)
-		(width 0.15)
-		(layer "B.Cu")
-		(net 5)
-	)
-	(segment
-		(start 141.5 66.5)
-		(end 141.5 71)
-		(width 0.15)
-		(layer "B.Cu")
-		(net 5)
-	)
-	(segment
-		(start 141.5 71)
-		(end 156 85.5)
-		(width 0.15)
-		(layer "B.Cu")
-		(net 5)
-	)
-	(segment
-		(start 156 90.5)
-		(end 147.5 99)
-		(width 0.15)
+		(width 0.2)
 		(layer "B.Cu")
 		(net 5)
@@
 	)
 	(segment
-		(start 156.3612 92.8612)
-		(end 156 92.5)
-		(width 0.15)
-		(layer "F.Cu")
-		(net 31)
-	)
-	(segment
-		(start 157.5422 92.8612)
-		(end 156.3612 92.8612)
-		(width 0.15)
-		(layer "F.Cu")
-		(net 31)
-	)
-	(segment
 		(start 157.821 67.2892)
 		(end 158.721 67.2892)
@@
 		(net 31)
 	)
-	(via
-		(at 156 92.5)
-		(size 0.6)
-		(drill 0.3)
-		(layers "F.Cu" "B.Cu")
+	(segment
+		(start 158.6682 91.7352)
+		(end 157.5422 92.8612)
+		(width 0.15)
+		(layer "B.Cu")
 		(net 31)
 	)
 	(segment
-		(start 158.6682 91.146004)
+		(start 159.071002 68.5)
 		(end 158.6682 68.902802)
 		(width 0.15)
@@
 	)
 	(segment
-		(start 156 92.5)
-		(end 157.314204 92.5)
-		(width 0.15)
-		(layer "B.Cu")
-		(net 31)
-	)
-	(segment
-		(start 157.314204 92.5)
-		(end 158.6682 91.146004)
-		(width 0.15)
-		(layer "B.Cu")
-		(net 31)
-	)
-	(segment
 		(start 158.6682 68.902802)
-		(end 159.071002 68.5)
-		(width 0.15)
-		(layer "B.Cu")
+		(end 158.6682 91.7352)
+		(width 0.15)
+		(layer "B.Cu")

Commit message: Final touchups and cleaned up layout
Routing:
- net /HX711 DOUT: track 103.9 -> 54.9 mm
- net /HX711 PDSCK: track 82.0 -> 54.2 mm, vias 2 -> 3
- net /LED: track 63.8 -> 47.5 mm, vias 2 -> 4
- net GND: track 13.4 -> 18.1 mm, vias 3 -> 5
- net +5V_USB: track 53.8 -> 49.5 mm, vias 6 -> 4
- net /BOOT: track 52.9 -> 51.4 mm, vias 1 -> 2
- net /RX: track 29.8 -> 30.0 mm, vias 0 -> 2
Other:
- board text added: "+"
- board text added: "-"
- board text added: "3.3V"
- board text added: "BATT 3.7V"
- board text added: "BOOT"
- board text added: "DOUT"
- board text added: "EN"
- board text added: "ESP-PROG"
- board text added: "GND"
- board text added: "HX711"
- board text added: "PDSCK"
- board text added: "Power REV5"
- board text added: "RX"
- board text added: "TX"
